File: D_Tympan_DFMI_1.0.kicad_pcb (KiCad board)
At the start: 4 copper layers, 38 x 74 mm, 116 parts, among them IC1 MK66FX1M0VMD18, IC2 MKL02Z32VFG4, IC3 BC127, J1 SJ-3523-SMT-TR, J2 SJ-3524-SMT-TR-PI, J3 alt Power Pads, P1 USB_OTG, P10 CONN_01X01, P2 CONN_01X06, P3 CONN_01X06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

Commit message: Added some notes on the PCB board file
This looks basically OK. I would 'soften' some of the traces where you have almost right angles in them, but that may be more asthetic. Please see the notes I have put on the Eco2.Use layer in the board file.
Other:
- board text added: "Make sure to include this annular ring in the GND net. You may need to draw a trace to connect it. Do the same for the other microphone"
Changed lines of the file:
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@@
-(kicad_pcb (version 20171130) (host pcbnew "(5.1.5)-3")
+(kicad_pcb (version 20171130) (host pcbnew "(5.1.4-0-10_14)")
   (general
     (thickness 1.6)
-    (drawings 86)
+    (drawings 89)
     (tracks 1615)
     (zones 0)
@@
   )
   (layers
-    (0 F.Cu signal)
+    (0 F.Cu signal hide)
     (1 In1.Cu signal)
-    (2 In2.Cu mixed)
+    (2 In2.Cu mixed hide)
     (31 B.Cu signal)
     (32 B.Adhes user)
     (33 F.Adhes user)
-    (34 B.Paste user hide)
+    (34 B.Paste user)
     (35 F.Paste user hide)
-    (36 B.SilkS user)
-    (37 F.SilkS user)
+    (36 B.SilkS user hide)
+    (37 F.SilkS user hide)
     (38 B.Mask user hide)
     (39 F.Mask user hide)
@@
     (41 Cmts.User user)
     (42 Eco1.User user hide)
-    (43 Eco2.User user hide)
+    (43 Eco2.User user)
     (44 Edge.Cuts user)
     (45 Margin user hide)
@@
   )
   (setup
-    (last_trace_width 0.1778)
+    (last_trace_width 0.25)
     (user_trace_width 0.1778)
     (user_trace_width 0.2032)
@@
     )
   )
+  (gr_line (start 117.35 64.48) (end 116.85 63.48) (layer Eco2.User) (width 0.15))
+  (gr_line (start 108.35 60.98) (end 117.35 64.48) (layer Eco2.User) (width 0.15))
+  (gr_text "Make sure to include this annular ring \nin the GND net.\nYou may need to draw a trace to connect it.\nDo the same for the other microphone" (at 94.85 56.98) (layer Eco2.User)
+    (effects (font (size 1 1) (thickness 0.15)))
+  )
   (gr_text "Dhwani 1.0\nUTSAAH Lab\nIISc" (at 133.05 52.73) (layer B.SilkS)

Commit message: final save on the changes
Other:
- board text added: "Concern that your copper pour on in2.C is not connected. Do a visual check. The 3V3 enters the board from this side (after the fuse) I’m not sure that you have the pour continuous. You can adjust the distance to the board edge, if that works with the DFM of your board house. Otherwise you may need to adjust traces."
- board text added: "Make sure to include this annular ring in the GND net. You may need to draw a trace to connect it. Do the same for the other microphone. They won’t be happy unless this connection is made"
- board text removed: "Make sure to include this annular ring in the GND net. You may need to draw a trace to connect it. Do the same for the other microphone"
Changed lines of the file:
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@@
   (general
     (thickness 1.6)
-    (drawings 89)
+    (drawings 90)
     (tracks 1615)
     (zones 0)
@@
   )
   (layers
-    (0 F.Cu signal hide)
-    (1 In1.Cu signal)
-    (2 In2.Cu mixed hide)
+    (0 F.Cu signal)
+    (1 In1.Cu signal hide)
+    (2 In2.Cu mixed)
     (31 B.Cu signal)
     (32 B.Adhes user)
@@
     )
   )
+  (gr_text "Concern that your copper pour on in2.C is not connected.\nDo a visual check. The 3V3 enters the board from this side (after the fuse)\nI’m not sure that you have the pour continuous. You can adjust the distance to the board edge,\nif that works with the DFM of your board house. Otherwise you may need to adjust traces." (at 109.35 101.48) (layer Eco2.User)
+    (effects (font (size 1 1) (thickness 0.15)) (justify right))
+  )
   (gr_line (start 117.35 64.48) (end 116.85 63.48) (layer Eco2.User) (width 0.15))
   (gr_line (start 108.35 60.98) (end 117.35 64.48) (layer Eco2.User) (width 0.15))
-  (gr_text "Make sure to include this annular ring \nin the GND net.\nYou may need to draw a trace to connect it.\nDo the same for the other microphone" (at 94.85 56.98) (layer Eco2.User)
-    (effects (font (size 1 1) (thickness 0.15)))
+  (gr_text "Make sure to include this annular ring in the GND net.\nYou may need to draw a trace to connect it.\nDo the same for the other microphone.\nThey won’t be happy unless this connection is made" (at 107.35 60.48) (layer Eco2.User)
+    (effects (font (size 1 1) (thickness 0.15)) (justify right))
   )
   (gr_text "Dhwani 1.0\nUTSAAH Lab\nIISc" (at 133.05 52.73) (layer B.SilkS)
